Commit message: refactor!: rename package to robot_rbvogui_base
Align package metadata, mesh URIs, documentation and tests with the base model identity.

BREAKING CHANGE: replace robot_rbvogui_common with robot_rbvogui_base, model_base.xacro with robot_rbvogui_base.xacro, and debug_model_base launch/script entry points with debug_robot_rbvogui_base.

File: urdf/basket/basket_macros.xacro (robot description, xacro)
@@ -7,15 +7,15 @@
   <xacro:include filename="$(find robotics_description)/urdf/common/all_commons.xacro"/>
   <xacro:property name="basket_chassis_visual_mesh"
-                  value="robot_rbvogui_common/meshes/basket/basket_container.obj"/>
+                  value="robot_rbvogui_base/meshes/basket/basket_container.obj"/>
   <xacro:property name="basket_chassis_collision_mesh"
-                  value="robot_rbvogui_common/meshes/basket/basket_container.stl"/>
+                  value="robot_rbvogui_base/meshes/basket/basket_container.stl"/>
   <xacro:property name="basket_chassis_closed_visual_mesh"
-                  value="robot_rbvogui_common/meshes/basket/basket_container.obj"/>
+                  value="robot_rbvogui_base/meshes/basket/basket_container.obj"/>
   <xacro:property name="basket_chassis_closed_collision_mesh"
-                  value="robot_rbvogui_common/meshes/basket/basket_container.stl"/>
+                  value="robot_rbvogui_base/meshes/basket/basket_container.stl"/>
   <xacro:property name="basket_sensors_visual_mesh"
-                  value="robot_rbvogui_common/meshes/basket/basket_sensors.obj"/>
+                  value="robot_rbvogui_base/meshes/basket/basket_sensors.obj"/>
   <xacro:property name="basket_sensors_collision_mesh"
-                  value="robot_rbvogui_common/meshes/basket/basket_sensors.stl"/>
+                  value="robot_rbvogui_base/meshes/basket/basket_sensors.stl"/>
   <!--
   Macro for the basket chassis.

File: urdf/common.xacro (robot description, xacro)
@@ -3,6 +3,7 @@
   <!--
   Shared RB-VOGUI mobile-base Xacro for four steerable wheels.
-  This file is not a complete robot model. Entry-point Xacros such as model_base.xacro and
-  model_forklift.xacro include it, then add their own links, sensors, actuators, and Gazebo plugins.
+  This file is not a complete robot model. Entry-point Xacros such as
+  robot_rbvogui_base.xacro and robot_rbvogui_forklift.xacro include it, then add their own links,
+  sensors, actuators, and Gazebo plugins.
   The base is composed of the RB-VOGUI chassis, battery and four steerable wheels:
   - Front-left wheel uses angle +alpha.
@@ -96,7 +97,7 @@
   <xacro:property name="battery_joint_origin"   value="0.02952 0 0 0 0 0"/>
   <xacro:property name="body_mesh_scale"        value="1.0 1.0 1.0"/>
-  <xacro:property name="chassis_visual_mesh"    value="robot_rbvogui_common/meshes/rbvogui_chassis.dae"/>
-  <xacro:property name="chassis_collision_mesh" value="robot_rbvogui_common/meshes/rbvogui_chassis.stl"/>
-  <xacro:property name="battery_mesh"           value="robot_rbvogui_common/meshes/rbvogui_battery.stl"/>
+  <xacro:property name="chassis_visual_mesh"    value="robot_rbvogui_base/meshes/rbvogui_chassis.dae"/>
+  <xacro:property name="chassis_collision_mesh" value="robot_rbvogui_base/meshes/rbvogui_chassis.stl"/>
+  <xacro:property name="battery_mesh"           value="robot_rbvogui_base/meshes/rbvogui_battery.stl"/>
   <xacro:property name="battery_color"
                   value="${robot_prefix}battery_color 0.08235 0.08235 0.08235 1.0"/>

File: urdf/robot_rbvogui_base.xacro (robot description, xacro)
@@ -2,8 +2,8 @@
 <robot name="rbvogui_base" xmlns:xacro="http://www.ros.org/wiki/xacro">
   <!--
-  This file publishes the `base` model of the `robot_rbvogui_common` family.
+  This file publishes the `base` model of the `robot_rbvogui_base` family.
   The robot name inside the URDF stays `rbvogui_base`.
   -->
-  <xacro:include filename="$(find robot_rbvogui_common)/urdf/common.xacro"/>
+  <xacro:include filename="$(find robot_rbvogui_base)/urdf/common.xacro"/>
   <!-- A non-empty sim_file adds the simulation-only joint-state publisher. -->
   <xacro:if value="${sim_file != ''}">
